File: tuck-n-roll/pcb/tuck-n-roll.kicad_pcb (KiCad board)
At the start: 2 copper layers, 154 x 101.8 mm, 62 parts

Commit message: Tuck n roll config update (#4)
Parts:
- removed the G*** at (8.13, 18.8)
- added D19: , ComboDiode, F.Cu at (64.4, 1.47)
- added HOLE1: , MountingHole_2.2mm_M2_Pad_Via, F.Cu at (85.2, -1.39)
- added HOLE2: , MountingHole_2.2mm_M2_Pad_Via, F.Cu at (87.9, -53.4)
- added HOLE3: , MountingHole_2.2mm_M2_Pad_Via, F.Cu at (3.98, -8.91)
- added HOLE4: , MountingHole_2.2mm_M2_Pad_Via, F.Cu at (-6.09, -42.8)
- added HOLE5: , MountingHole_2.2mm_M2_Pad_Via, F.Cu at (44.6, -47.4)
- G***: value LOGO -> FRONTLOGOSILK
- moved S5 0.20 mm to (-16.6, -31.2)
- moved S6 0.20 mm to (-16.6, -31.2)
- moved D9 0.20 mm to (39.9, -55.2)
- moved S17 0.20 mm to (31.7, -54.4)
- moved S18 0.20 mm to (31.7, -54.4)
- moved D12 0.20 mm to (64.6, -53.4)
- moved D15 0.20 mm to (83.6, -52.4)
- moved MCU1 0.20 mm to (103.3, -44.4)
- moved S23 0.20 mm to (56.3, -53.4)
- moved S24 0.20 mm to (56.3, -53.4)
- moved S29 0.20 mm to (75.3, -52.4)
- moved S30 0.20 mm to (75.3, -52.4)
- moved D6 0.20 mm to (13.3, -51.3)
- moved S11 0.20 mm to (5.29, -49.2)
- moved S12 0.20 mm to (5.29, -49.2)
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Connections:
- REF** pad C: P14 -> GND
- REF** pad D: P15 -> (no net)
- REF** pad S2: GND -> enc_diode
Routing:
- net P15: track 87.6 -> 0.00 mm
- net P14: track 81.5 -> 0.00 mm
- net P21: track 189.5 -> 228.9 mm
- net enc_diode: track 0.00 -> 17.0 mm
- net P7: track 92.7 -> 109.3 mm
- net GND: track 0.00 -> 11.2 mm
- net P6: track 375.6 -> 374.1 mm
Other:
- board size 154 x 101.8 mm -> 154 x 101.6 mm

Commit message: Update tuck-n-roll to latest version
Parts:
- added B1: SW_RST, TACT_SWITCH_TVBP06, F.Cu at (118.3, -42.4)
Routing:
- net RST: track 0.00 -> 25.7 mm
